Commit message: feat: add differential drive and validate robot motion

File: src/robot_description/urdf/amr.urdf.xacro (robot description, xacro)
@@ -49,5 +49,5 @@
             <origin xyz="0 0 0.10"
                     rpy="0 0 0"/>
-            <mass value="15.0"/>    # 무게(kg)
+            <mass value="15.0"/>
             <inertia
                 ixx="0.25"
@@ -97,5 +97,5 @@
         <origin xyz="0 0.22 0"
                 rpy="1.5708 0 0"/>
-        <axis xyz="0 0 1"/>
+        <axis xyz="0 0 -1"/>
     </joint>
     <gazebo reference="left_wheel_link">
@@ -139,5 +139,5 @@
         <origin xyz="0 -0.22 0"
                 rpy="1.5708 0 0"/>
-        <axis xyz="0 0 1"/>
+        <axis xyz="0 0 -1"/>
     </joint>
     <gazebo reference="right_wheel_link">
@@ -263,3 +263,18 @@
     <mu2>0.01</mu2>
     </gazebo>
+    <!-- ========================= -->
+    <!-- DIFFERENTIAL DRIVE -->
+    <!-- ========================= -->
+    <gazebo>
+        <plugin
+            filename="ignition-gazebo-diff-drive-system"
+            name="ignition::gazebo::systems::DiffDrive">
+            <left_joint>left_wheel_joint</left_joint>
+            <right_joint>right_wheel_joint</right_joint>
+            <wheel_separation>0.44</wheel_separation>
+            <wheel_radius>0.08</wheel_radius>
+            <topic>cmd_vel</topic>
+            <odom_publish_frequency>50</odom_publish_frequency>
+        </plugin>
+    </gazebo>
 </robot>
